File: 01_MultichannelUniversalDAQ/DAQ_PCB_Frontend_Bridge_DS_ADC_v1.0/DAQ_PCB_Frontend_Bridge_DS_ADC_v1.0.kicad_sch (KiCad schematic)
At the start: 6 parts

Commit message: bugfix
Connections:
- net GND: now reaches H3.1
- net GND: now also H1.1, H2.1, H4.1, H5.1, H6.1
- no-connect marks 10 -> 4
