File: 01_MultichannelUniversalDAQ/DAQ_PCB_Frontend_Universal_SAR_ADC_v1.0/DAQ_PCB_Frontend_Universal_SAR_ADC_v1.0.kicad_pcb (KiCad board)
At the start: 2 copper layers, 384 parts, among them J2 Conn_01x05, J3 Conn_01x05, J4 Conn_01x05, J5 Conn_01x05, J6 Conn_01x05, J7 Conn_01x05, J8 Conn_01x05, J9 Conn_01x05, U1 24AA02E, U10 LT3092, U11 INA823, U12 LT3092, U13 INA823, U14 LT3092, U15 INA823, U16 LT3092, U17 INA823, U18 LT3092, U19 INA823, U2 LT3092, U20 LT3092, U21 INA823, U22 TLA2518, U3 INA823, U4 OPA2197, U5 OPA2197, U6 OPA2197, U7 OPA2197, U8 LT3092, U9 INA823

Commit message: 0. placement concept (SAR_ADC)
Parts:
- added R213: 0R, Resistor_SMD:R_0603_1608Metric_Pad0.98x0.95mm_HandSolder, F.Cu at (60.7, 71.8)
- added R214: 0R, Resistor_SMD:R_0603_1608Metric_Pad0.98x0.95mm_HandSolder, F.Cu at (64.4, 76.0)
- added R215: 0R, Resistor_SMD:R_0603_1608Metric_Pad0.98x0.95mm_HandSolder, F.Cu at (57.5, 71.8)
- added R216: 0R, Resistor_SMD:R_0603_1608Metric_Pad0.98x0.95mm_HandSolder, F.Cu at (59.1, 71.8)
- added R217: 0R, Resistor_SMD:R_0603_1608Metric_Pad0.98x0.95mm_HandSolder, F.Cu at (62.3, 71.8)
- added R218: 0R, Resistor_SMD:R_0603_1608Metric_Pad0.98x0.95mm_HandSolder, F.Cu at (66.0, 76.0)
- added U23: MCP3208, Package_SO:SOIC-16_3.9x9.9mm_P1.27mm, B.Cu at (59.8, 78.1)
- C2, C20, C21, C27, C28, C3, C34, C35, C41, C42, C48, C49, C55, C56, C63, C65, D1, D3, D4, D5, D6, D7, D8, R100, R101, R102, R112, R12, R124, R125, R126, R127, R137, R149, R150, R151, R152, R162, R174, R175, R176, R177, R187, R199, R200, R201, R202, R24, R25, R26, R27, R62, R74, R75, R76, R77, R87, R99: moved to B.Cu
- moved R26 155.9 mm to (81.6, 97.0), turned to 90 degrees
- moved D1 155.5 mm to (75.9, 94.0), turned to 180 degrees
- moved R27 154.9 mm to (81.6, 91.1), turned to 90 degrees
- moved TP22 154.1 mm to (88.3, 96.8)
- moved TP23 152.7 mm to (88.3, 91.4)
- moved C2 148.7 mm to (85.4, 95.1), turned to 180 degrees
- moved C3 148.0 mm to (85.4, 93.1), turned to 180 degrees
- moved R21 147.4 mm to (91.8, 101.0), turned to 90 degrees
- moved C4 144.8 mm to (88.4, 94.1), turned to 90 degrees
- moved R23 144.1 mm to (94.8, 101.9)
- moved J2 144.0 mm to (79.1, 87.7), turned to -90 degrees
- moved R29 143.5 mm to (85.4, 91.1), turned to 180 degrees
- moved C6 143.0 mm to (90.1, 98.4), turned to 90 degrees
- moved R30 142.8 mm to (85.4, 89.0), turned to 180 degrees
- moved TP24 142.3 mm to (99.8, 100.4)
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Connections:
- U22 pad 11: /ADC/ADC_SPI.CSn -> Net-(U22-~{CS})
- U22 pad 13: /ADC/ADC_SPI.SCK -> Net-(U22-CLK)
- U22 pad 14: /ADC/ADC_SPI.MOSI -> Net-(U22-SDI)
Routing:
- net Net-(U23-Din): track 0.00 -> 2.26 mm, vias 0 -> 1
- net Net-(U23-Dout): track 0.00 -> 2.07 mm
Other:
- board outline added: 60 x 110.1 mm

Commit message: 0. placement concept (SAR_ADC)
Parts:
- C19, C26, C33, C40, C47, C54, C61, C8, R109, R110, R134, R135, R159, R160, R184, R185, R209, R210, R34, R35, R59, R60, R84, R85: moved to B.Cu
- moved TP35 5.00 mm to (72.0, 95.4)
- moved TP38 5.00 mm to (72.0, 115.4)
- moved TP41 5.00 mm to (100.0, 115.4)
- moved TP44 5.00 mm to (72.0, 139.4)
- moved TP47 5.00 mm to (100.0, 139.4)
- moved TP50 5.00 mm to (72.0, 159.4)
- moved TP53 5.00 mm to (100.0, 159.4)
- moved TP24 5.00 mm to (100.0, 95.4)
- moved C19 4.00 mm to (69.8, 95.7)
- moved C40 4.00 mm to (69.8, 139.7)
- moved C47 4.00 mm to (97.8, 139.7)
- moved C54 4.00 mm to (69.8, 159.7)
- moved C61 4.00 mm to (97.8, 159.7)
- moved C26 4.00 mm to (69.8, 115.7)
- moved C33 4.00 mm to (97.8, 115.7)
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Other:
- board size 60 x 110.1 mm -> 60 x 110 mm
