File: 01_MultichannelUniversalDAQ/DAQ_PCB_Frontend_Universal_SAR_ADC_v1.0/ADC_SAR.kicad_sch (KiCad schematic)
At the start: 9 parts, among them U22 TLA2518, U23 MCP3208

Commit message: 0. placement concept (SAR_ADC)
Parts:
- added R213, R214, R215, R216, R217, R218: 0R, Resistor_SMD:R_0603_1608Metric_Pad0.98x0.95mm_HandSolder, symbol Device:R_Small
- U23: footprint (none) -> Package_SO:SOIC-16_3.9x9.9mm_P1.27mm
Connections:
- net ADC_SPI.CSn: now also R214.2, R218.2; no longer U22.11 (~{CS}), U23.10 (~{CS}/SHDN)
- net ADC_SPI.MOSI: now also R213.2, R217.2; no longer U22.14 (SDI), U23.11 (Din)
- net ADC_SPI.SCK: now also R215.2, R216.2; no longer U22.13 (CLK), U23.13 (CLK)
- new net: R213.1, U22.14 (SDI)
- new net: R216.1, U23.13 (CLK)
- new net: R214.1, U22.11 (~{CS})
- new net: R215.1, U22.13 (CLK)
- new net: R217.1, U23.11 (Din)
- new net: R218.1, U23.10 (~{CS}/SHDN)

Commit message: Commit after meeting
Other:
- note added: "ADC: ADAS3022 +-15V táp: LTC3260"
Changed lines of the file:
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@@
 		(comment 3 "16 Channel Data Acquisition (DAQ) Board")
+	)
+	(text "ADC: ADAS3022\n+-15V táp: LTC3260\n"
+		(exclude_from_sim no)
+		(at 145.288 31.496 0)
+		(effects
+			(font
+				(size 2.54 2.54)
+				(thickness 0.508)
+				(bold yes)
+				(color 255 0 0 1)
+			)
+		)
 	)
 	(text "Alternative ADC option"

Commit message: ADC és preamp in progress
Parts:
- removed C62, C63, C66: 1u, Capacitor_SMD:C_0603_1608Metric_Pad1.08x0.95mm_HandSolder, symbol Device:C_Small
- removed C64, C65: 100n, Capacitor_SMD:C_0603_1608Metric_Pad1.08x0.95mm_HandSolder, symbol Device:C_Small
- removed R211, R212: 33R, Resistor_SMD:R_0603_1608Metric_Pad0.98x0.95mm_HandSolder, symbol Device:R_Small
- removed R213, R214, R215, R216, R217, R218: 0R, Resistor_SMD:R_0603_1608Metric_Pad0.98x0.95mm_HandSolder, symbol Device:R_Small
- removed U22: TLA2518, Package_DFN_QFN:WQFN-16-1EP_3x3mm_P0.5mm_EP1.6x1.6mm, symbol KJ_KiCadLib:TLA2518
- removed U23: MCP3208, Package_SO:SOIC-16_3.9x9.9mm_P1.27mm, symbol Analog_ADC:MCP3208
Other:
- note removed: "ADC"
- note removed: "ADC: ADAS3022 +-15V táp: LTC3260"
- note removed: "Alternative ADC option"
