File: 01_MultichannelUniversalDAQ/DAQ_PCB_Frontend_Universal_SAR_ADC_v1.0/AnalogFrontend.kicad_sch (KiCad schematic)
At the start: 16 parts, among them U4 OPA2197, U5 OPA2197, U6 OPA2197, U7 OPA2197

Commit message: ...
Parts:
- removed C10, C11, C12, C9: 100n, Capacitor_SMD:C_0603_1608Metric_Pad1.08x0.95mm_HandSolder, symbol Device:C_Small
- removed TP25, TP26, TP27, TP28, TP29, TP30, TP31, TP32: TestPoint, TestPoint:TestPoint_Pad_D1.0mm, symbol Connector:TestPoint
- removed U4, U5, U6, U7: OPA2197, Package_SO:SOIC-8_3.9x4.9mm_P1.27mm, symbol Amplifier_Operational:OPA2197xD
Other:
- sheet PREAMP1 ports: added +12V, +15V, +24V, +5V, -15V; removed 10V, 2V5, 5V, VCC+, VCC-
- sheet PREAMP2 ports: added +12V, +15V, +24V, +5V, -15V; removed 10V, 2V5, 5V, VCC+, VCC-
- sheet PREAMP3 ports: added +12V, +15V, +24V, +5V, -15V; removed 10V, 2V5, 5V, VCC+, VCC-
- sheet PREAMP4 ports: added +12V, +15V, +24V, +5V, -15V; removed 10V, 2V5, 5V, VCC+, VCC-
- sheet PREAMP5 ports: added +12V, +15V, +24V, +5V, -15V; removed 10V, 2V5, 5V, VCC+, VCC-
- sheet PREAMP6 ports: added +12V, +15V, +24V, +5V, -15V; removed 10V, 2V5, 5V, VCC+, VCC-
- sheet PREAMP7 ports: added +12V, +15V, +24V, +5V, -15V; removed 10V, 2V5, 5V, VCC+, VCC-
- sheet PREAMP8 ports: added +12V, +15V, +24V, +5V, -15V; removed 10V, 2V5, 5V, VCC+, VCC-
- note removed: "5V Related signal"
- note removed: "Multifunctional Voltage or Current Measurement"
- note removed: "Output Buffer"
- note removed: "PreAmp Channels"
