File: 01_MultichannelUniversalDAQ/DAQ_PCB_MainBoard_v1.0/DAQ_PCB_MainBoard_v1.0.kicad_sch (KiCad schematic)
At the start: 7 parts

Commit message: bugfix
Other:
- sheet PWR ports: added PWR_SENSE; removed PWR_MEAS
Changed lines of the file:
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@@
-			)
-		)
-		(pin "PWR_MEAS" output
-			(at 146.05 63.5 270)
-			(effects
-				(font
-					(size 1.27 1.27)
-				)
-				(justify left)
 			)
 		)
@@
 			(effects
 				(font
+					(size 1.27 1.27)
+				)
+				(justify left)
+			)
+		)
+		(pin "PWR_SENSE" output
+			(at 146.05 63.5 270)
+			(effects
+				(font

Commit message: Commit after meeting
Other:
- note added: "https://www.tme.eu/hu/details/g3127/univerzalis-keszulekhazak/gainta/"
Changed lines of the file:
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@@
+		)
+	)
+	(text "https://www.tme.eu/hu/details/g3127/univerzalis-keszulekhazak/gainta/"
+		(exclude_from_sim no)
+		(at 84.074 191.77 0)
+		(effects
+			(font
+				(size 1.27 1.27)
+			)
 		)
 	)
