File: 01_MultichannelUniversalDAQ/DAQ_PCB_MainBoard_v1.0/DAQ_PCB_MainBoard_v1.0.kicad_pcb (KiCad board)
At the start: 2 copper layers, 250 parts, among them J1 Molex 1x2, J10 Molex 1x3, J12 Conn_02x13_Row_Letter_Last_Mo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, J13 Conn_01x02, J2 Pin Header 1x6, J5 2.54 mm Header, J6 2.54 mm Header, J7 USB_B_Micro, Q1 SQ2337CES, Q2 SQ2337CES, U1 REF5050, U10 MCP9700Ax-ELT, U11 STM32-H563ZI, U12 USBLC6-2SC6, U13 LAN8742AI, U14 USBLC6-2SC6, U15 USBLC6-2SC6, U2 NCV8182C, U3 NCV8182C, U4 NCV8182C, U5 DPBW06, U6 SPBW06, U7 INA823, U9 TPS22919, Y2 32.768kHz

Commit message: Commit after meeting
Parts:
- added J11: 7499211121A, KJ_KiCadLib_Others_Footprint:T_Wurth_WE-RJ45LAN_7499211121A, F.Cu at (211.8, 76.7)
- added J3: ~, KJ_KiCadLib_Others_Footprint:15210502601000, F.Cu at (170.4, 42.7)
- added J4: ~, KJ_KiCadLib_Others_Footprint:15210502601000, F.Cu at (170.4, 55.2)
- added L7: MPZ2012S601AT000, Inductor_SMD:L_0805_2012Metric_Pad1.05x1.20mm_HandSolder, F.Cu at (172.5, 63.8)
- moved J10 161.9 mm to (211.5, 87.0)
- moved J6 161.5 mm to (216.1, 95.2)
- moved J5 161.5 mm to (211.5, 95.2)
- moved J7 160.8 mm to (224.0, 96.0)
- moved J1 159.6 mm to (220.5, 87.0)
- moved U6 157.8 mm to (220.0, 53.0)
- moved U5 157.8 mm to (220.0, 40.0)
- moved J13 120.8 mm to (227.5, 87.0)
- renumbered U17 to J12
Connections:
- C39 pad 1: /PWR/PWR_SENSE.BATT -> /MCU/PWR_SENSE.BATT
- H2 pad 1: MGND -> unconnected-(H2-Pad1)
- H3 pad 1: MGND -> unconnected-(H3-Pad1)_2
- H4 pad 1: MGND -> unconnected-(H4-Pad1)_2
- R31 pad 1: /PWR/PWR_SENSE.BATT -> /MCU/PWR_SENSE.BATT
- R32 pad 1: /PWR/PWR_SENSE.BATT -> /MCU/PWR_SENSE.BATT
- R41 pad 1: Net-(R33-Pad2) -> -12V
- TP8 pad 1: /PWR/PWR_SENSE.BATT -> /MCU/PWR_SENSE.BATT
- U11 pad 114: unconnected-(U11-PD0-Pad114) -> /DIGI_IO/ID.0
- U11 pad 115: unconnected-(U11-PD1-Pad115) -> /DIGI_IO/ID.1
- U11 pad 116: unconnected-(U11-PD2-Pad116) -> /DIGI_IO/ID.2
- U11 pad 123: unconnected-(U11-PD7-Pad123) -> /DIGI_IO/ID.3

Commit message: Power meas
Parts:
- moved C24 144.6 mm to (225.2, 33.7)
Changed lines of the file:
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@@
 	(footprint "Capacitor_SMD:C_0603_1608Metric_Pad1.08x0.95mm_HandSolder"
 		(layer "F.Cu")
-		(at 80.8234 41.9954)
+		(at 225.2 33.7)
 		(descr "Capacitor SMD 0603 (1608 Metric), square (rectangular) end terminal, IPC-7351 nominal with elongated pad for handsoldering. (Body size source: IPC-SM-782 page 76, https://www.pcb-3d.com/wordpress/wp-content/uploads/ipc-sm-782a_amendment_1_and_2.pdf)")
 		(tags "capacitor handsolder")
