File: 01_MultichannelUniversalDAQ/DAQ_PCB_MainBoard_v1.0/PWR_Sup.kicad_sch (KiCad schematic)
At the start: 10 parts, among them U8 LM2901

Commit message: Power meas
Parts:
- added R95, R96: 10k, Resistor_SMD:R_0603_1608Metric_Pad0.98x0.95mm_HandSolder, symbol Device:R_Small
- R34: value 33k -> 120k
- R36: value 33k -> 82k
- R37: value 47k -> 10k
- R38: value 33k -> 51k
- R39: value 12k -> 10k
- R40: value 10k -> 18k
- R41: value 160k -> 10k
Connections:
- net -12V_SEN is gone; now on net GND: R41.1
- net 5V_PG is gone; now on net 16V5_PG: U8.1
- net 3V3: now also R95.2; no longer R40.2
- net 5V_SEN: now also R40.2; no longer R36.2
- net GND: now also R96.1
- net at R40.1, R41.2: now also U8.9 (+); no longer U8.8 (-)
- net +12V_PG renamed 24V_PG
- net +12V_SEN renamed 24V_SEN
- net -12V_PG renamed 16V5_PG
- net 10V_PG renamed 12V_PG
- net 10V_SEN renamed 12_SEN
- net 2V5_REF: no longer names the net of U8.10 (-), U8.4 (-), U8.6 (-)
- net 2V5_REF: now also U8.8 (-), R95.1, R96.2; no longer U8.9 (+)
- new net 16V5_SEN: R36.2
Other:
- note added: "TH = 10.1V"
- note added: "TH = 15.2V"
- note added: "TH = 21.5V"
- note added: "TH = 4.62V"
- note removed: "TH = -10.3V or 2V5ref fault"
- note removed: "TH = 10.75V"
- note removed: "TH = 4.25V"
- note removed: "TH = 9.4V"
- moved on the sheet: C40, R40, R41, U8E
