File: 01_MultichannelUniversalDAQ/DAQ_PCB_MainBoard_v1.0/EthernetPHY.kicad_sch (KiCad schematic)
At the start: 39 parts, among them J11 7499211121A, U13 LAN8742AI, U14 USBLC6-2SC6, U15 USBLC6-2SC6, Y3 25MHz

Commit message: bugfix
Parts:
- J11: footprint Transformer_THT_Wurth:T_Wurth_WE-RJ45LAN_7499211121A -> KJ_KiCadLib_Others_Footprint:T_Wurth_WE-RJ45LAN_7499211121A
- L7: footprint Inductor_SMD:L_0805_2012Metric_Pad1.15x1.40mm_HandSolder -> Inductor_SMD:L_0805_2012Metric_Pad1.05x1.20mm_HandSolder
Changed lines of the file:
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@@
 			)
 		)
-		(property "Footprint" "Inductor_SMD:L_0805_2012Metric_Pad1.15x1.40mm_HandSolder"
+		(property "Footprint" "Inductor_SMD:L_0805_2012Metric_Pad1.05x1.20mm_HandSolder"
 			(at 85.09 130.81 0)
 			(hide yes)
@@
 			)
 		)
-		(property "Footprint" "Transformer_THT_Wurth:T_Wurth_WE-RJ45LAN_7499211121A"
+		(property "Footprint" "KJ_KiCadLib_Others_Footprint:T_Wurth_WE-RJ45LAN_7499211121A"
 			(at 254 49.53 0)
 			(hide yes)

Commit message: new power concept
Parts:
- removed C77: 470n, Capacitor_SMD:C_1206_3216Metric_Pad1.33x1.80mm_HandSolder, symbol Device:C_Small
- added C9: 1u, Capacitor_SMD:C_1206_3216Metric_Pad1.33x1.80mm_HandSolder, symbol Device:C_Small
- added D9: SMAJ58CA, Diode_SMD:D_SMA, symbol Diode:SMAJ24CA
- added R97: 0R, Resistor_SMD:R_1206_3216Metric_Pad1.30x1.75mm_HandSolder, symbol Device:R_Small
Connections:
- net VCC_PoE+: now also C9.1, D9.2 (A2)
- net VCC_PoE-: now also C9.2, D9.1 (A1), R97.2
- net at J11.S1 (SHIELD1), J11.S2 (SHIELD2), R89.2: now also R97.1
