File: 01_MultichannelUniversalDAQ/DAQ_PCB_MainBoard_v1.0/Power.kicad_sch (KiCad schematic)
At the start: 98 parts, among them J1 Molex 1x2, J14 Pin Header 1x5, Q1 SQ2337CES, Q2 SQ2337CES, U1 REF5050, U19 SPBW06, U20 LMR51630Y, U21 LMR51630Y, U3 NCV8182C, U5 DPBW06, U6 SPBW06

Commit message: Power meas
Other:
- sheet Power Supervisor ports: added 12V_PG, 12_SEN, 16V5_PG, 16V5_SEN, 24V_PG, 24V_SEN; removed +12V_PG, +12V_SEN, -12V_PG, -12V_SEN, 10V_PG, 10V_SEN, 2V5_REF
- note added: "acc.: 0.05% real / 0.25% w.c."
- note removed: "acc.: 0.03% real / 0.2% w.c."
Changed lines of the file:
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@@
 		)
 	)
-	(text "acc.: 0.03% real / 0.2% w.c."
+	(text "acc.: 0.05% real / 0.25% w.c."
 		(exclude_from_sim no)
 		(at 214.63 192.786 0)
@@
 	(wire
 		(pts
-			(xy 314.96 182.88) (xy 321.31 182.88)
-		)
-		(stroke
-			(width 0)
-			(type default)
-		)
-	)
-	(wire
-		(pts
 			(xy 148.59 57.15) (xy 163.83 57.15)
 		)
@@
 	(wire
 		(pts
+			(xy 187.96 158.75) (xy 187.96 201.93)
+		)
+		(stroke
+			(width 0)
+			(type default)
+		)
+	)
+	(wire
+		(pts
 			(xy 365.76 133.35) (xy 365.76 128.27)
 		)
@@
 	(wire
 		(pts
+			(xy 104.14 158.75) (xy 187.96 158.75)
+		)
+		(stroke
+			(width 0)
+			(type default)
+		)
+	)
+	(wire
+		(pts
 			(xy 163.83 200.66) (xy 163.83 205.74)
 		)
@@
 	(wire
 		(pts
-			(xy 187.96 196.85) (xy 187.96 201.93)
-		)
-		(stroke
-			(width 0)
-			(type default)
-		)
-	)
-	(wire
-		(pts
 			(xy 198.12 81.28) (xy 213.36 81.28)
 		)
@@
 	)
 	(image
-		(at 139.446 164.846)
+		(at 270.256 268.986)
 		(scale 0.470616)
 		(data "iVBORw0KGgoAAAANSUhEUgAABPMAAAI7CAYAAACJC95NAAAABHNCSVQICAgIfAhkiAAAIABJREFU"
@@
 		)
 	)
-	(label "PWR_SENSE{+12V 10V 5V -12V BATT}"
+	(label "PWR_SENSE{24V 16V5 12V 5V BATT}"
 		(at 381 199.39 90)
 		(effects
@@
 		)
 	)
-	(label "PWR_SENSE.5V"
+	(label "PWR_SENSE.12V"
 		(at 360.68 191.77 0)
 		(effects
@@
 		)
 	)
-	(label "PWR_SENSE.+12V"
+	(label "PWR_SENSE.24V"
 		(at 360.68 186.69 0)
 		(effects
@@
 		)
 	)
-	(label "PWR_SENSE.10V"
+	(label "PWR_SENSE.16V5"
 		(at 360.68 189.23 0)
 		(effects
@@
 		)
 	)
-	(label "PWR_SENSE.-12V"
+	(label "PWR_SENSE.5V"
 		(at 360.68 194.31 0)
 		(effects
@@
 			)
 		)
-		(property "Value" "-12V"
-			(at 309.626 194.31 90)
+		(property "Value" "5V"
+			(at 310.134 194.31 90)
 			(show_name no)
 			(do_not_autoplace no)
@@
 			)
 		)
-		(property "Value" "5V"
+		(property "Value" "12V"
 			(at 310.134 191.77 90)
 			(show_name no)
@@
 			)
 		)
-		(property "Value" "+12V"
+		(property "Value" "24V"
 			(at 309.626 186.69 90)
 			(show_name no)
@@
 	)
 	(symbol
-		(lib_id "power:VCC")
-		(at 187.96 196.85 0)
-		(unit 1)
-		(body_style 1)
-		(exclude_from_sim no)
-		(in_bom yes)
-		(on_board yes)
-		(in_pos_files yes)
-		(dnp no)
-		(property "Reference" "#PWR046"
-			(at 187.96 200.66 0)
-			(hide yes)
-			(show_name no)
-			(do_not_autoplace no)
-			(effects
-				(font
-					(size 1.27 1.27)
-				)
-			)
-		)
-		(property "Value" "5Vref"
-			(at 187.96 193.294 0)
-			(show_name no)
-			(do_not_autoplace no)
-			(effects
-				(font
-					(size 1.27 1.27)
-				)
-			)
-		)
-		(property "Footprint" ""
-			(at 187.96 196.85 0)
-			(hide yes)
-			(show_name no)
-			(do_not_autoplace no)
-			(effects
-				(font
-					(size 1.27 1.27)
-				)
-			)
-		)
-		(property "Datasheet" ""
-			(at 187.96 196.85 0)
-			(hide yes)
-			(show_name no)
-			(do_not_autoplace no)
-			(effects
-				(font
-					(size 1.27 1.27)
-				)
-			)
-		)
-		(property "Description" "Power symbol creates a global label with name \"VCC\""
-			(at 187.96 196.85 0)
-			(hide yes)
-			(show_name no)
-			(do_not_autoplace no)
-			(effects
-				(font
-					(size 1.27 1.27)
-				)
-			)
-		)
-		(pin "1"
-		)
-		(instances
-			(project "DAQ_PCB_MainBoard_v1.0"
-				(path "/4059b195-d7bb-4a1b-a7b6-e8bbfebcd311/10176249-18d5-40a7-abbb-e6394fe2f254"
-					(reference "#PWR046")
-					(unit 1)
-				)
-			)
-		)
-	)
-	(symbol
 		(lib_id "power:GNDA")
 		(at 130.81 265.43 0)
@@
 			)
 		)
-		(property "Value" "+10V"
+		(property "Value" "16V5"
 			(at 309.626 189.23 90)
 			(show_name no)
@@
 	)
 	(symbol
-		(lib_id "power:VCC")
-		(at 314.96 182.88 90)
-		(unit 1)
-		(body_style 1)
-		(exclude_from_sim no)
-		(in_bom yes)
-		(on_board yes)
-		(in_pos_files yes)
-		(dnp no)
-		(property "Reference" "#PWR074"
-			(at 318.77 182.88 0)
-			(hide yes)
-			(show_name no)
-			(do_not_autoplace no)
-			(effects
-				(font
-					(size 1.27 1.27)
-				)
-			)
-		)
-		(property "Value" "2V5ref"
-			(at 308.864 182.88 90)
-			(show_name no)
-			(do_not_autoplace no)
-			(effects
-				(font
-					(size 1.27 1.27)
-				)
-			)
-		)
-		(property "Footprint" ""
-			(at 314.96 182.88 0)
-			(hide yes)
-			(show_name no)
-			(do_not_autoplace no)
-			(effects
-				(font
-					(size 1.27 1.27)
-				)
-			)
-		)
-		(property "Datasheet" ""
-			(at 314.96 182.88 0)
-			(hide yes)
-			(show_name no)
-			(do_not_autoplace no)
-			(effects
-				(font
-					(size 1.27 1.27)
-				)
-			)
-		)
-		(property "Description" "Power symbol creates a global label with name \"VCC\""
-			(at 314.96 182.88 0)
-			(hide yes)
-			(show_name no)
-			(do_not_autoplace no)
-			(effects
-				(font
-					(size 1.27 1.27)
-				)
-			)
-		)
-		(pin "1"
-		)
-		(instances
-			(project "DAQ_PCB_MainBoard_v1.0"
-				(path "/4059b195-d7bb-4a1b-a7b6-e8bbfebcd311/10176249-18d5-40a7-abbb-e6394fe2f254"
-					(reference "#PWR074")
-					(unit 1)
-				)
-			)
-		)
-	)
-	(symbol
 		(lib_id "Device:C_Small")
 		(at 215.9 81.28 90)
@@
 			)
 		)
-		(pin "2V5_REF" input
-			(at 321.31 182.88 180)
-			(effects
-				(font
-					(size 1.27 1.27)
-				)
-				(justify left)
-			)
-		)
 		(pin "VCC" input
 			(at 321.31 180.34 180)
@@
 			)
 		)
-		(pin "+12V_PG" output
-			(at 351.79 186.69 0)
+		(pin "5V_PG" output
+			(at 351.79 194.31 0)
 			(effects
 				(font
@@
 			)
 		)
-		(pin "+12V_SEN" input
-			(at 321.31 186.69 180)
+		(pin "5V_SEN" input
+			(at 321.31 194.31 180)
 			(effects
 				(font
@@
 			)
 		)
-		(pin "-12V_PG" output
-			(at 351.79 194.31 0)
+		(pin "12V_PG" output
+			(at 351.79 191.77 0)
 			(effects
 				(font
@@
 			)
 		)
-		(pin "-12V_SEN" input
-			(at 321.31 194.31 180)
+		(pin "12_SEN" input
+			(at 321.31 191.77 180)
 			(effects
 				(font
@@
 			)
 		)
-		(pin "5V_PG" output
-			(at 351.79 191.77 0)
+		(pin "16V5_PG" output
+			(at 351.79 189.23 0)
 			(effects
 				(font
@@
 			)
 		)
-		(pin "5V_SEN" input
-			(at 321.31 191.77 180)
+		(pin "16V5_SEN" input
+			(at 321.31 189.23 180)
 			(effects
 				(font
@@
 			)
 		)
-		(pin "10V_SEN" input
-			(at 321.31 189.23 180)
+		(pin "24V_PG" output
+			(at 351.79 186.69 0)
 			(effects
 				(font
 					(size 1.27 1.27)
 				)
-				(justify left)
+				(justify right)
 			)
 		)
-		(pin "10V_PG" output
-			(at 351.79 189.23 0)
+		(pin "24V_SEN" input
+			(at 321.31 186.69 180)
 			(effects
 				(font
 					(size 1.27 1.27)
 				)
-				(justify right)
+				(justify left)
 			)
 		)

Commit message: new power concept
Parts:
- removed C1, C4: 2u2, Capacitor_SMD:C_0805_2012Metric_Pad1.18x1.45mm_HandSolder, symbol Device:C_Small
- removed C18, C19, C31: 470n, Capacitor_SMD:C_1206_3216Metric_Pad1.33x1.80mm_HandSolder, symbol Device:C_Small
- removed R7: 1k5, Resistor_SMD:R_0603_1608Metric_Pad0.98x0.95mm_HandSolder, symbol Device:R_Small
- added C102, C111: 1u, Capacitor_SMD:C_0603_1608Metric_Pad1.08x0.95mm_HandSolder, symbol Device:C_Small
- added C6, C7, C8: 1u, Capacitor_SMD:C_1206_3216Metric_Pad1.33x1.80mm_HandSolder, symbol Device:C_Small
- C3, C5: value 470n -> 1u; Part Number C1206C474KMREC7210 -> CL31B105KCHNNNE; Voltage 63V -> 100V
- D1: value SMAJ60CA -> SMAJ48CA
- R25: value 1k -> 1k5
- R33: value 4k7 -> 6k8
Connections:
- net +12V: now also C111.1
- net 5Vref: now also C102.1
- net GND: now also C102.2, C111.2
- net VBAT_CON-: now also C8.2; no longer C5.2
- net VIN+: now also C5.1, C6.1, C7.1
- net VIN-: now also C5.2, C6.2, C7.2
- net VIN_UNFILT+: now also C8.1; no longer C5.1
Other:
- sheet Battery Measurement ports: added DIAG, SGN_OUT+, SGN_OUT-; removed SGN_OUT
- moved on the sheet: C100, C101, C2, C20, C21, C22, C23, C24, C25, C26, C27, C28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
