File: 01_MultichannelUniversalDAQ/DAQ_PCB_MainBoard_v1.0/STM32-H563.kicad_sch (KiCad schematic)
At the start: 79 parts, among them J10 Molex 1x3, J5 2.54 mm Header, J6 2.54 mm Header, J7 USB_B_Micro, J8 Pin Header, J9 Pin Header, U10 MCP9700Ax-ELT, U11 STM32-H563ZI, U12 USBLC6-2SC6, U9 TPS22919, Y1 25MHz, Y2 32.768kHz

Commit message: bugfix
Connections:
- no-connect marks 23 -> 24

Commit message: new power concept
Parts:
- removed C41, C43: 100n, Capacitor_SMD:C_0603_1608Metric_Pad1.08x0.95mm_HandSolder, symbol Device:C_Small
- removed R42: 33k, Resistor_SMD:R_0603_1608Metric_Pad0.98x0.95mm_HandSolder, symbol Device:R_Small
- removed R43: 12k, Resistor_SMD:R_0603_1608Metric_Pad0.98x0.95mm_HandSolder, symbol Device:R_Small
- removed R47, R50: 0R, Resistor_SMD:R_0603_1608Metric_Pad0.98x0.95mm_HandSolder, symbol Device:R_Small
- removed U9: TPS22919, Package_TO_SOT_SMD:SOT-363_SC-70-6, symbol KJ_KiCadLib:TPS22919
- added C112, C113, C12: 1u, Capacitor_SMD:C_0603_1608Metric_Pad1.08x0.95mm_HandSolder, symbol Device:C_Small
- added C77: 100n, Capacitor_SMD:C_0603_1608Metric_Pad1.08x0.95mm_HandSolder, symbol Device:C_Small
- added R107, R108: 0R, Resistor_SMD:R_0603_1608Metric_Pad0.98x0.95mm_HandSolder, symbol Device:R_Small
- added TP27, TP8: TestPoint, TestPoint:TestPoint_Pad_D1.0mm, symbol Connector:TestPoint
- added U2: REF5025, Package_SO:SOIC-8_3.9x4.9mm_P1.27mm, symbol Reference_Voltage:REF5025AD
- D6: value LED_RED -> LED_GREEN
- R46: value 0R -> 10k; now fitted
Connections:
- net PWR_SENSE.-12V is gone; now on net PWR_SENSE.5V: U11.21 (PF9)
- net 3V3: now also C113.1, R108.2, U2.2 (Vin); no longer R46.2
- net GND: now also R46.2, C112.2, C113.2, C12.2, C77.2, U2.4 (GND)
- net MCU_VREF: now also C77.1, R107.1, R108.1, TP27.1
- net PWR_SENSE.5V: no longer U11.20 (PF8)
- net PWR_SENSE.BATT_N: now reaches U11.50 (PF12)
- net PWR_SENSE.BATT_DIAG: now reaches U11.55 (PF15)
- net PWR_SENSE.+12V renamed PWR_SENSE.24V
- net PWR_SENSE.10V renamed PWR_SENSE.16V5
- net PWR_SENSE.BATT renamed PWR_SENSE.BATT_P
- new net: C12.1, U2.5 (Trim/NR)
- new net: C112.1, R107.2, U2.6 (Vout)
- new net: TP8.1, U2.3 (Temp)
- new net PWR_SENSE.12V: U11.20 (PF8)
- no-connect marks 24 -> 23
Other:
- note added: "2V5 REF @10mA"
- note removed: "MCU ADC Vref"
- note removed: "PWR Switch: VREF ON if 3V3"
